File: HF/kicad/modulation_HF/modulation_HF.kicad_sch (KiCad schematic)
At the start: 0 parts

Commit message: filtre en ordre 2+ passage en alternatif+ ajout sur kicad + ajout kicad interrupteur pour piloter l'entré/ sortie de l'antenne. manque plus que le gain en sortie du mélangeure
Parts:
- added C1, C7: 100p, symbol Device:C
- added C10: 1n, symbol Device:C
- added C11, C3, C6: 10n, symbol Device:C
- added C12, C14: 1µ, symbol Device:C
- added C13, C2, C4, C8: 10p, symbol Device:C
- added C15: 10µF, symbol Device:C
- added C5: 470p, symbol Device:C
- added C9: 2p, symbol Device:C
- added J1: Conn_01x05_Pin, symbol Connector:Conn_01x05_Pin
- added J3: Conn_Coaxial, symbol Connector:Conn_Coaxial
- added R1, R8: 220k, symbol Device:R
- added R10: 5600, symbol Device:R
- added R11, R3: 150, symbol Device:R
- added R12, R14, R5: 1k, symbol Device:R
- added R13, R4: 1,2k, symbol Device:R
- added R15, R16: 470, symbol Device:R
- added R2, R7: 11M, symbol Device:R
- added R6: 560, symbol Device:R
- added R9: 10k, symbol Device:R
- added U1, U4: ~, symbol Projet personelle:CD74HC4046AE
- added U2, U3: ADE-6, RF_Mini-Circuits:Mini-Circuits_CD542_LandPatternPL-052, symbol RF_Mixer:ADE-6
- added U5, U7: 74HCT00, symbol 74xx:74HCT00
- added U6: MASW-007221, Package_TO_SOT_SMD:SOT-363_SC-70-6, symbol RF_Switch:MASW-007221
- added Y1: 13,56Mhz, symbol Device:Crystal
Connections:
- new net: C3.1, R11.1, R3.2
- new net: C15.2, R16.1, U5.4, U5.5
- new net: R15.1, U5.1, U5.2, Y1.1
- new net: C15.1, R15.2, U5.3
- new net: C4.1, R13.1, R4.2
- new net: C11.1, C12.1, R11.2
- new net: R1.1, U1.11 (R1)
- new net: C13.1, C14.1, R13.2
- new net: J3.1 (In), U6.5 (RFC)
- new net: C6.2, R5.2, R6.2
- new net: R8.1, U4.11 (R1)
- new net: R7.1, U4.12 (R2)
- new net: R9.2, U4.2 (PC1out)
- new net: U4.3 (COMPin), U4.4 (VCOout)
- new net: C7.1, U4.6 (C1A)
- new net: C7.2, U4.7 (C1B)
- new net: R2.1, U1.12 (R2)
- new net: C1.1, U1.6 (C1A)
- new net: C1.2, U1.7 (C1B)
- new net +5V: C2.1, C8.1, J1.2 (Pin_2), U1.16 (VCC), U4.16 (VCC)
- new net GND: C10.2, C11.2, C13.2, C2.2, C3.2, C4.2, C5.2, C8.2, C9.2, J1.1 (Pin_1), J3.2 (Ext), R1.2, R12.2, R14.2, R2.2, R6.1, R7.2, R8.2, U1.8 (GND), U2.1 (GND), U2.4 (GND), U2.5 (GND), U3.1 (GND), U3.4 (GND), U3.5 (GND), U4.8 (GND)
- new net Oscilateur: R16.2, R4.1, U3.6 (LO), U5.6, Y1.2
- new net OscilateurFiltré: C14.2, R14.1, U2.6 (LO)
- new net SignalDémel: C6.1, U3.2 (IF)
- new net SignalFiltré: C5.1, R5.1, U4.14 (SIGin)
- new net SignalRecus: U3.3 (RF), U6.1 (RF1)
- new net SignalàEnvoyer: U2.2 (IF), U6.3 (RF2)
- new net VCOin: J1.3 (Pin_3), U1.9 (VCOin)
- new net VCOout: R3.1, U1.4 (VCOout)
- new net VCOoutFiltré: C12.2, R12.1, U2.3 (RF)
- new net ctrl_Sortie_Antenne: J1.5 (Pin_5), U6.4 (V2), U7.1, U7.2
- new net signal vers µc: C10.1, J1.4 (Pin_4), R10.1
- new net signalDemodul: C9.1, R10.2, R9.1, U4.9 (VCOin)
- new net ~{ctrl_Sortie_Antenne}: U6.6 (V1), U7.3
- no-connect marks 0 -> 13
Other:
- note added: "Connecteurs"
- note added: "Filtres"
- note added: "VCO et PLL"
- note added: "mélangeur HF"
