File: HF/kicad/Adaptation antenne/Adaptation antenne.kicad_sch (KiCad schematic)
At the start: 6 parts, among them J1 Conn_Coaxial, J2 Impédence Antenne, J3 impédence GND, J4 Sortie vers antenne, J5 Sortie vers GND, J6 Antenne

Commit message: modif kicad pour ajusté au test sur platin
Other:
- title: (none) -> Adaptateur antenne vers bnc 
Changed lines of the file:
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@@
 	(generator_version "9.0")
 	(paper "A4")
+	(title_block
+		(title "Adaptateur antenne vers bnc ")
+		(date "2026-03-27")
+	)
 	(junction
 		(at 40.64 24.13)
